File: Digital-PA-Push-Pull-Final-v2/digital-amp.kicad_pcb (KiCad board)
At the start: 2 copper layers, 93.5 x 65.5 mm, 56 parts, among them J1 FAN, K1 Omron G5V-2 / OEN 46-05-2C, Q1 AOD407, Q2 2N3904, Q3 IRF510, Q4 IRF510, Q5 2N3904, T1 BN-43-3312, 1T+1T:3T, U2 L7812, U6 L7805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

Commit message: A new beginning...
Parts:
- added C17: 1n, Capacitor_SMD:C_1206_3216Metric_Pad1.33x1.80mm_HandSolder, F.Cu at (108.3, 57.0)
- added C18: 10n, Capacitor_SMD:C_1206_3216Metric_Pad1.33x1.80mm_HandSolder, F.Cu at (108.3, 59.5)
- C16: value 1n -> 10n
Routing:
- net +VDC: track 52.0 -> 61.3 mm
- net GND: vias 286 -> 282
