File: Digital-PA-Push-Pull-Final-v2/digital-amp.kicad_sch (KiCad schematic)
At the start: 56 parts, among them J1 FAN, K1 Omron G5V-2 / OEN 46-05-2C, Q1 AOD407, Q2 2N3904, Q3 IRF510, Q4 IRF510, Q7 2N3904, T1 BN-43-3312, 1T+1T:3T, U2 L7812, U6 L7805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

Commit message: A new beginning...
Parts:
- added C17: 1n, Capacitor_SMD:C_1206_3216Metric_Pad1.33x1.80mm_HandSolder, symbol Device:C_Small
- added C18: 10n, Capacitor_SMD:C_1206_3216Metric_Pad1.33x1.80mm_HandSolder, symbol Device:C_Small
- C16: value 1n -> 10n
Connections:
- net +VDC: now also C17.1, C18.1
- net GND: now also C17.2, C18.2
Changed lines of the file:
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@@
 	)
 	(junction
+		(at 218.44 67.31)
+		(diameter 0)
+		(color 0 0 0 0)
+	)
+	(junction
 		(at 170.18 44.45)
 		(diameter 0)
@@
 	)
 	(junction
+		(at 223.52 67.31)
+		(diameter 0)
+		(color 0 0 0 0)
+	)
+	(junction
 		(at 38.1 175.26)
 		(diameter 0)
@@
 	)
 	(junction
+		(at 228.6 72.39)
+		(diameter 0)
+		(color 0 0 0 0)
+	)
+	(junction
 		(at 182.88 102.87)
 		(diameter 0)
@@
 		(color 0 0 0 0)
 	)
+	(junction
+		(at 223.52 72.39)
+		(diameter 0)
+		(color 0 0 0 0)
+	)
 	(no_connect
 		(at 107.95 154.94)
@@
 	(wire
 		(pts
-			(xy 198.12 67.31) (xy 228.6 67.31)
+			(xy 198.12 67.31) (xy 218.44 67.31)
 		)
 		(stroke
@@
 	(wire
 		(pts
+			(xy 218.44 67.31) (xy 223.52 67.31)
+		)
+		(stroke
+			(width 0)
+			(type default)
+		)
+	)
+	(wire
+		(pts
+			(xy 223.52 72.39) (xy 228.6 72.39)
+		)
+		(stroke
+			(width 0)
+			(type default)
+		)
+	)
+	(wire
+		(pts
 			(xy 238.76 67.31) (xy 254 67.31)
 		)
@@
 	(wire
 		(pts
-			(xy 233.68 72.39) (xy 233.68 74.93)
-		)
-		(stroke
-			(width 0)
-			(type default)
-		)
-	)
-	(wire
-		(pts
 			(xy 167.64 44.45) (xy 170.18 44.45)
 		)
@@
 	(wire
 		(pts
+			(xy 218.44 72.39) (xy 223.52 72.39)
+		)
+		(stroke
+			(width 0)
+			(type default)
+		)
+	)
+	(wire
+		(pts
 			(xy 50.8 62.23) (xy 52.07 62.23)
 		)
@@
 	(wire
 		(pts
+			(xy 223.52 67.31) (xy 228.6 67.31)
+		)
+		(stroke
+			(width 0)
+			(type default)
+		)
+	)
+	(wire
+		(pts
 			(xy 223.52 45.72) (xy 223.52 46.99)
 		)
@@
 			)
 		)
-		(property "Value" "1n"
+		(property "Value" "10n"
 			(at 233.934 71.374 0)
 			(effects
@@
 	)
 	(symbol
+		(lib_id "Device:C_Small")
+		(at 223.52 69.85 0)
+		(unit 1)
+		(exclude_from_sim no)
+		(in_bom yes)
+		(on_board yes)
+		(dnp no)
+		(property "Reference" "C18"
+			(at 223.774 68.072 0)
+			(effects
+				(font
+					(size 0.9906 0.9906)
+				)
+				(justify left)
+			)
+		)
+		(property "Value" "10n"
+			(at 223.774 71.374 0)
+			(effects
+				(font
+					(size 0.9906 0.9906)
+				)
+				(justify left)
+			)
+		)
+		(property "Footprint" "Capacitor_SMD:C_1206_3216Metric_Pad1.33x1.80mm_HandSolder"
+			(at 223.52 69.85 0)
+			(effects
+				(font
+					(size 1.27 1.27)
+				)
+				(hide yes)
+			)
+		)
+		(property "Datasheet" "~"
+			(at 223.52 69.85 0)
+			(effects
+				(font
+					(size 1.27 1.27)
+				)
+				(hide yes)
+			)
+		)
+		(property "Description" ""
+			(at 223.52 69.85 0)
+			(effects
+				(font
+					(size 1.27 1.27)
+				)
+				(hide yes)
+			)
+		)
+		(property "Ext" "HV"
+			(at 223.52 69.85 0)
+			(effects
+				(font
+					(size 1.524 1.524)
+				)
+				(hide yes)
+			)
+		)
+		(pin "1"
+		)
+		(pin "2"
+		)
+		(instances
+			(project "digital-amp"
+				(path "/816a895b-d385-40fc-87bf-7154a813d474"
+					(reference "C18")
+					(unit 1)
+				)
+			)
+		)
+	)
+	(symbol
 		(lib_id "power:GND")
 		(at 67.31 165.1 0)
@@
 	(symbol
 		(lib_id "power:GND")
-		(at 233.68 74.93 0)
+		(at 228.6 72.39 0)
 		(unit 1)
 		(exclude_from_sim no)
@@
 		(dnp no)
 		(property "Reference" "#PWR054"
-			(at 233.68 81.28 0)
+			(at 228.6 78.74 0)
 			(effects
 				(font
@@
 		)
 		(property "Value" "GND"
-			(at 233.68 78.74 0)
+			(at 228.6 76.2 0)
 			(effects
 				(font
@@
 		)
 		(property "Footprint" ""
-			(at 233.68 74.93 0)
+			(at 228.6 72.39 0)
 			(effects
 				(font
@@
 		)
 		(property "Datasheet" ""
-			(at 233.68 74.93 0)
+			(at 228.6 72.39 0)
 			(effects
 				(font
@@
 		)
 		(property "Description" ""
-			(at 233.68 74.93 0)
+			(at 228.6 72.39 0)
 			(effects
 				(font
@@
 					(unit 1)
 				)
+			)
+		)
+	)
+	(symbol
+		(lib_id "Device:C_Small")
+		(at 218.44 69.85 0)
+		(unit 1)
+		(exclude_from_sim no)
+		(in_bom yes)
+		(on_board yes)
+		(dnp no)
+		(property "Reference" "C17"
+			(at 218.694 68.072 0)
+			(effects
+				(font
+					(size 0.9906 0.9906)
+				)
+				(justify left)
+			)
+		)
+		(property "Value" "1n"
+			(at 218.694 71.628 0)
+			(effects
+				(font
+					(size 0.9906 0.9906)
+				)
+				(justify left)
+			)
+		)
+		(property "Footprint" "Capacitor_SMD:C_1206_3216Metric_Pad1.33x1.80mm_HandSolder"
+			(at 218.44 69.85 0)
+			(effects
+				(font
+					(size 1.27 1.27)
+				)
+				(hide yes)
+			)
+		)
+		(property "Datasheet" "~"
+			(at 218.44 69.85 0)
+			(effects
+				(font
+					(size 1.27 1.27)
+				)
+				(hide yes)
+			)
+		)
+		(property "Description" ""
+			(at 218.44 69.85 0)
+			(effects
+				(font
+					(size 1.27 1.27)
+				)
+				(hide yes)
+			)
+		)
+		(property "Ext" "HV"
+			(at 218.44 69.85 0)
+			(effects
+				(font
+					(size 1.524 1.524)
+				)
+				(hide yes)
+			)
+		)
+		(pin "1"
+		)
+		(pin "2"
+		)
+		(instances
+			(project "digital-amp"
+				(path "/816a895b-d385-40fc-87bf-7154a813d474"
+					(reference "C17")
+					(unit 1)
+				)
