File: DDX-1-R2.20/DDX-1-R2.20.kicad_pcb (KiCad board)
At the start: 2 copper layers, 90 x 99.9 mm, 101 parts, among them K1 HFD4/5-S, Q1 2N3904, Q2 IRF510, Q5 SS9018, T1 Bifilar XFMR, U1 L7805, U2 UCC27517ADBVR, U3 L7809, U4 LD1117S33CTR, U5 SI5351_Module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

Commit message: Changes from Windows PC
Parts:
- U3: value L7809 -> LM7809_TO220; footprint footprints:TO-252-2-Longer -> footprints:TO-220-3_Horizontal_TabDown
- moved TP2 51.2 mm to (166.8, 154.4)
- moved U3 27.7 mm to (151.3, 70.2), turned to 180 degrees
- moved C32 22.8 mm to (152.8, 65.5), turned to 0 degrees
- moved D1 21.3 mm to (173.2, 70.5), turned to 180 degrees
- moved U1 20.8 mm to (157.2, 103.4)
- moved C1 13.0 mm to (146.2, 65.5)
- moved C9 9.71 mm to (145.6, 103.0), turned to 90 degrees
- moved C14 9.48 mm to (166.9, 106.0)
- moved D5 4.48 mm to (142.6, 108.8)
- moved C11 2.77 mm to (179.1, 71.2)
- moved C17 2.77 mm to (185.3, 71.2)
- moved C6 2.77 mm to (188.1, 71.2)
- moved C10 2.77 mm to (181.9, 71.2)
- moved L4 2.39 mm to (138.9, 104.4)
- moved C44 2.09 mm to (141.7, 100.6), turned to 90 degrees
Connections:
- C1 pad 1: 12V -> +9V
- U1 pad 1: 12V -> +9V
Routing:
- net +9V: track 105.5 -> 171.3 mm
- net 12V: track 134.3 -> 87.7 mm, vias 0 -> 4
- net GND: track 167.7 -> 179.7 mm, vias 184 -> 183
- net Net-(U1-OUT): track 27.5 -> 18.3 mm
- net Net-(D5-K): track 44.0 -> 37.8 mm
- net +VDC: track 9.54 -> 6.79 mm
Other:
- outline, holes or cut-outs redrawn
- board text added: "GDS"
