File: DDX-1-R2.20/DDX-1-R2.20.kicad_sch (KiCad schematic)
At the start: 101 parts, among them K1 HFD4/5-S, Q2 IRF510, Q5 SS9018, Q7 2N3904, T1 Bifilar XFMR, U1 CD2003GB_GP, U1 L7805, U2 MCP6002, U2 UCC27517ADBVR, U3 L7809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

Commit message: Changes from Windows PC
Parts:
- removed U3: L7809, footprints:TO-252-2-Longer, symbol Regulator_Linear:L7809
- added U3: LM7809_TO220, footprints:TO-220-3_Horizontal_TabDown, symbol Regulator_Linear:LM7809_TO220
Connections:
- net +9V: now also C1.1, U1.1 (IN), U3.3 (VO)
- net 12V: now also U3.1 (VI); no longer C1.1, U1.1 (IN)
- net GND: now also U3.2 (GND)
Other:
- note removed: "DPAK"
Changed lines of the file:
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@@
 		)
 	)
-	(text "DPAK"
-		(exclude_from_sim no)
-		(at 223.266 54.864 0)
-		(effects
-			(font
-				(size 1.27 1.27)
-			)
-		)
-	)
 	(text "T/R switch (with RX grounding)"
 		(exclude_from_sim no)
@@
 	)
 	(junction
-		(at 187.96 22.86)
-		(diameter 0)
-		(color 0 0 0 0)
-	)
-	(junction
 		(at 111.76 185.42)
 		(diameter 0)
@@
 	)
 	(junction
-		(at 236.22 22.86)
+		(at 208.28 203.2)
 		(diameter 0)
 		(color 0 0 0 0)
 	)
 	(junction
-		(at 208.28 203.2)
+		(at 182.88 88.9)
 		(diameter 0)
 		(color 0 0 0 0)
 	)
 	(junction
-		(at 182.88 88.9)
+		(at 187.96 22.86)
 		(diameter 0)
 		(color 0 0 0 0)
@@
 	(wire
 		(pts
-			(xy 236.22 20.32) (xy 236.22 22.86)
+			(xy 236.22 20.32) (xy 236.22 58.42)
 		)
 		(stroke
@@
 	(wire
 		(pts
+			(xy 187.96 22.86) (xy 193.04 22.86)
+		)
+		(stroke
+			(width 0)
+			(type default)
+		)
+	)
+	(wire
+		(pts
 			(xy 200.66 203.2) (xy 200.66 208.28)
 		)
@@
 	(wire
 		(pts
-			(xy 236.22 58.42) (xy 236.22 22.86)
-		)
-		(stroke
-			(width 0)
-			(type default)
-		)
-	)
-	(wire
-		(pts
 			(xy 187.96 88.9) (xy 203.2 88.9)
 		)
@@
 	(wire
 		(pts
-			(xy 187.96 22.86) (xy 236.22 22.86)
-		)
-		(stroke
-			(width 0)
-			(type default)
-		)
-	)
-	(wire
-		(pts
 			(xy 186.69 309.88) (xy 190.5 309.88)
 		)
@@
 	)
 	(symbol
+		(lib_id "power:+9V")
+		(at 193.04 22.86 0)
+		(unit 1)
+		(exclude_from_sim no)
+		(in_bom yes)
+		(on_board yes)
+		(dnp no)
+		(fields_autoplaced yes)
+		(property "Reference" "#PWR043"
+			(at 193.04 26.67 0)
+			(effects
+				(font
+					(size 1.27 1.27)
+				)
+				(hide yes)
+			)
+		)
+		(property "Value" "+9V"
+			(at 193.04 17.78 0)
+			(effects
+				(font
+					(size 1.27 1.27)
+				)
+			)
+		)
+		(property "Footprint" ""
+			(at 193.04 22.86 0)
+			(effects
+				(font
+					(size 1.27 1.27)
+				)
+				(hide yes)
+			)
+		)
+		(property "Datasheet" ""
+			(at 193.04 22.86 0)
+			(effects
+				(font
+					(size 1.27 1.27)
+				)
+				(hide yes)
+			)
+		)
+		(property "Description" "Power symbol creates a global label with name \"+9V\""
+			(at 193.04 22.86 0)
+			(effects
+				(font
+					(size 1.27 1.27)
+				)
+				(hide yes)
+			)
+		)
+		(pin "1"
+		)
+		(instances
+			(project "DDX-1-R2.20"
+				(path "/cb614b23-9af3-4aec-bed8-c1374e001510"
+					(reference "#PWR043")
+					(unit 1)
+				)
+			)
+		)
+	)
+	(symbol
 		(lib_id "power:+5V")
 		(at 76.2 33.02 0)
@@
 	)
 	(symbol
-		(lib_id "Regulator_Linear:L7809")
-		(at 217.17 58.42 0)
-		(mirror y)
-		(unit 1)
-		(exclude_from_sim no)
-		(in_bom yes)
-		(on_board yes)
-		(dnp no)
-		(property "Reference" "U3"
-			(at 212.598 64.77 0)
-			(effects
-				(font
-					(size 1.27 1.27)
-				)
-			)
-		)
-		(property "Value" "L7809"
-			(at 217.17 54.61 0)
-			(effects
-				(font
-					(size 1.27 1.27)
-				)
-			)
-		)
-		(property "Footprint" "footprints:TO-252-2-Longer"
-			(at 216.535 62.23 0)
-			(effects
-				(font
-					(size 1.27 1.27)
-					(italic yes)
-				)
-				(justify left)
-				(hide yes)
-			)
-		)
-		(property "Datasheet" "http://www.st.com/content/ccc/resource/technical/document/datasheet/41/4f/b3/b0/12/d4/47/88/CD00000444.pdf/files/CD00000444.pdf/jcr:content/translations/en.CD00000444.pdf"
-			(at 217.17 59.69 0)
-			(effects
-				(font
-					(size 1.27 1.27)
-				)
-				(hide yes)
-			)
-		)
-		(property "Description" "Positive 1.5A 35V Linear Regulator, Fixed Output 9V, TO-220/TO-263/TO-252"
-			(at 217.17 58.42 0)
-			(effects
-				(font
-					(size 1.27 1.27)
-				)
-				(hide yes)
-			)
-		)
-		(pin "2"
-		)
-		(pin "1"
-		)
-		(pin "3"
-		)
-		(instances
-			(project ""
-				(path "/cb614b23-9af3-4aec-bed8-c1374e001510"
-					(reference "U3")
-					(unit 1)
-				)
-			)
-		)
-	)
-	(symbol
 		(lib_id "power:GND")
 		(at 186.69 314.96 0)
@@
 					(unit 1)
 				)
+			)
+		)
+	)
+	(symbol
+		(lib_id "Regulator_Linear:LM7809_TO220")
+		(at 217.17 58.42 0)
+		(mirror y)
+		(unit 1)
+		(exclude_from_sim no)
+		(in_bom yes)
+		(on_board yes)
+		(dnp no)
+		(property "Reference" "U3"
+			(at 217.17 52.07 0)
+			(effects
+				(font
+					(size 1.27 1.27)
+				)
+			)
+		)
+		(property "Value" "LM7809_TO220"
+			(at 217.17 54.61 0)
+			(effects
+				(font
+					(size 1.27 1.27)
+				)
+			)
+		)
+		(property "Footprint" "footprints:TO-220-3_Horizontal_TabDown"
+			(at 217.17 52.705 0)
+			(effects
+				(font
+					(size 1.27 1.27)
+					(italic yes)
+				)
+				(hide yes)
+			)
+		)
+		(property "Datasheet" "https://www.onsemi.cn/PowerSolutions/document/MC7800-D.PDF"
+			(at 217.17 59.69 0)
+			(effects
+				(font
+					(size 1.27 1.27)
+				)
+				(hide yes)
+			)
+		)
+		(property "Description" "Positive 1A 35V Linear Regulator, Fixed Output 9V, TO-220"
+			(at 217.17 58.42 0)
+			(effects
+				(font
+					(size 1.27 1.27)
+				)
+				(hide yes)
+			)
+		)
+		(pin "1"
+		)
+		(pin "3"
+		)
+		(pin "2"
+		)
+		(instances
+			(project ""
+				(path "/cb614b23-9af3-4aec-bed8-c1374e001510"
+					(reference "U3")
+					(unit 1)
+				)
