File: RX-TX-BPF-2025-v2/TX-BPF.kicad_pcb (KiCad board)
At the start: 11 copper layers, 62 x 28.6 mm, 21 parts

Commit message: New projects...
Routing:
- net Net-(CSL1-Pad1): track 18.7 -> 24.4 mm
- net Net-(OUT1-In): track 11.1 -> 7.15 mm
- net GND: track 58.6 -> 57.3 mm, vias 37 -> 33
- net Net-(CSS1-Pad1): track 6.51 -> 7.69 mm
- net Net-(CFS1-Pad2): track 5.44 -> 6.57 mm
- net Net-(CFL1-Pad1): track 17.0 -> 17.7 mm
- net Net-(CTS1-Pad1): track 8.66 -> 9.17 mm
Other:
- board text added: "TX-BPF Yantra Research © 2024"
- board text removed: "Yantra Research TX-BPF 2024 (C)"
