File: Easy-QRP-LPF-2025-v1/QRP-LPF.kicad_sch (KiCad schematic)
At the start: 21 parts

Commit message: Work on CWX
Parts:
- removed CFS1, CSL1, CSL3, CSS2, CTS1: 100n, Capacitor_SMD:C_1206_3216Metric_Pad1.33x1.80mm_HandSolder, symbol Device:C_Small
- removed CFS2, CSL2, CSS1, CTS2: 100n, Capacitor_SMD:C_1812_4532Metric_Pad1.57x3.40mm_HandSolder, symbol Device:C_Small
- added C1: 100n, Capacitor_SMD:C_0805_2012Metric_Pad1.18x1.45mm_HandSolder, symbol Device:C_Small
- C2: renamed from CFL1; footprint Capacitor_SMD:C_1206_3216Metric_Pad1.33x1.80mm_HandSolder -> Capacitor_SMD:C_0805_2012Metric_Pad1.18x1.45mm_HandSolder
- C3: renamed from CFL2; footprint Capacitor_SMD:C_1206_3216Metric_Pad1.33x1.80mm_HandSolder -> Capacitor_SMD:C_0805_2012Metric_Pad1.18x1.45mm_HandSolder
- C4: renamed from CFL3; footprint Capacitor_SMD:C_1812_4532Metric_Pad1.57x3.40mm_HandSolder -> Capacitor_SMD:C_0805_2012Metric_Pad1.18x1.45mm_HandSolder
- L1, L2, L3: footprint footprints:T50-6 -> Inductor_SMD:L_0805_2012Metric_Pad1.05x1.20mm_HandSolder
Connections:
- net GND: now also C1.2
- net at C2.1, L2.1: now also L1.2; no longer C3.1, C4.1
- net at IN1.1 (In), L1.1: now also C1.1
- net at L3.1: now also C3.1, L2.2
- net at L3.2: now also C4.1, OUT1.1 (In)
Other:
- note added: "Topology design by Elsie"
- note removed: "Topology: Mesh capacitor-coupled bandpass (Elsie)"
- moved on the sheet: IN1, L1, OUT1
